File: kicad/LDR_Night_Lamp/LDR_Night_Lamp.kicad_sch (KiCad schematic)
At the start: 0 parts

Commit message: feat: implement LDR night lamp schematic
Parts:
- added BT1: 9V, symbol Device:Battery
- added D1: LED, symbol Device:LED
- added Q1: BC547, Package_TO_SOT_THT:TO-92_Inline, symbol Transistor_BJT:BC547
- added R1: 100k, symbol Device:R
- added R2: LDR07, OptoDevice:R_LDR_5.1x4.3mm_P3.4mm_Vertical, symbol Sensor_Optical:LDR07
- added R3: 470R, symbol Device:R
Connections:
- new net: BT1.1 (+), R1.2, R3.1
- new net: D1.2 (A), R3.2
- new net: D1.1 (K), Q1.1 (C)
- new net: Q1.2 (B), R1.1, R2.1
- new net: BT1.2 (-), Q1.3 (E), R2.2
Other:
- title: (none) -> LDR Night Lamp

Commit message: feat: assigned footprints to schematic components
Parts:
- BT1: footprint (none) -> Battery:BatteryHolder_MPD_BA9VPC_1xPP3
- D1: footprint (none) -> LED_THT:LED_D5.0mm
- R1, R3: footprint (none) -> Resistor_THT:R_Axial_DIN0207_L6.3mm_D2.5mm_P15.24mm_Horizontal
Changed lines of the file:
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@@
 			)
 		)
-		(property "Footprint" ""
+		(property "Footprint" "Resistor_THT:R_Axial_DIN0207_L6.3mm_D2.5mm_P15.24mm_Horizontal"
 			(at 163.322 57.15 90)
 			(effects
@@
 			)
 		)
-		(property "Footprint" ""
+		(property "Footprint" "LED_THT:LED_D5.0mm"
 			(at 165.1 71.12 0)
 			(effects
@@
 			)
 		)
-		(property "Footprint" ""
+		(property "Footprint" "Resistor_THT:R_Axial_DIN0207_L6.3mm_D2.5mm_P15.24mm_Horizontal"
 			(at 144.018 58.42 90)
 			(effects
@@
 			)
 		)
-		(property "Footprint" ""
+		(property "Footprint" "Battery:BatteryHolder_MPD_BA9VPC_1xPP3"
 			(at 115.57 65.786 90)
 			(effects
