File: kicad/LDR_Night_Lamp/LDR_Night_Lamp.kicad_pcb (KiCad board)
At the start: 2 copper layers, 68.5 x 39 mm, 6 parts, among them Q1 BC547

Commit message: feat: added PCB silkscreen graphics and board markings
Parts:
- added G***: LOGO, LOGO, F.Cu at (115.0, 97.5)
- added REF**: WEEE-Logo_4.2x6mm_SilkScreen, Symbol:WEEE-Logo_4.2x6mm_SilkScreen, B.Cu at (143.0, 89.5)
- added REF**: KiCad-Logo2_5mm_SilkScreen, Symbol:KiCad-Logo2_5mm_SilkScreen, B.Cu at (143.0, 74.0)
- added REF**: OSHW-Logo_7.5x8mm_SilkScreen, Symbol:OSHW-Logo_7.5x8mm_SilkScreen, B.Cu at (143.0, 82.0)
- moved D1 15.3 mm to (176.0, 83.6)
- moved Q1 15.3 mm to (176.0, 90.6)
- moved R1 15.3 mm to (174.0, 77.2)
- moved R2 15.3 mm to (175.5, 96.1)
- moved BT1 15.3 mm to (117.2, 70.9)
- moved R3 15.3 mm to (178.0, 77.2)
Other:
- board text added: "SHARULE"
